File: kicad/keyboard/keyboard.kicad_pcb (KiCad board)
At the start: 2 copper layers, 244 x 92 mm, 119 parts, among them SW1 SW_MX, SW10 SW_MX, SW11 SW_MX, SW12 SW_MX, SW13 SW_MX, SW14 SW_MX, SW15 SW_MX, SW16 SW_MX, SW17 SW_MX, SW18 SW_MX, SW19 SW_MX, SW2 SW_MX, SW20 SW_MX, SW21 SW_MX, SW22 SW_MX, SW23 SW_MX, SW24 SW_MX, SW25 SW_MX, SW26 SW_MX, SW27 SW_MX, SW28 SW_MX, SW29 SW_MX, SW3 SW_MX, SW30 SW_MX, SW31 SW_MX, SW32 SW_MX, SW33 SW_MX, SW34 SW_MX, SW35 SW_MX, SW36 SW_MX, SW37 SW_MX, SW38 SW_MX, SW39 SW_MX, SW4 SW_MX, SW40 SW_MX, SW41 SW_MX, SW42 SW_MX, SW43 SW_MX, SW44 SW_MX, SW45 SW_MX, SW46 SW_MX, SW47 SW_MX, SW48 SW_MX, SW49 SW_MX, SW5 SW_MX, SW50 SW_MX, SW51 SW_MX, SW52 SW_MX, SW53 SW_MX, SW54 SW_MX, SW55 SW_MX, SW56 SW_MX, SW57 SW_MX, SW58 SW_MX, SW59 SW_MX, SW6 SW_MX, SW7 SW_MX, SW8 SW_MX, SW9 SW_MX

Commit message: Connect rows and columns to Pico
Parts:
- moved A1 0.26 mm to (248.6, 54.7)
Connections:
- A1 pad 1: COL0 -> ROW4
- A1 pad 10: COL6 -> ROW3
- A1 pad 11: ROW3 -> COL6
- A1 pad 17: unconnected-(A1-GPIO13-Pad17) -> ROW2
- A1 pad 19: ROW2 -> unconnected-(A1-GPIO14-Pad19)
- A1 pad 2: COL1 -> COL0
- A1 pad 20: unconnected-(A1-GPIO15-Pad20) -> COL11
- A1 pad 24: COL11 -> COL12
- A1 pad 25: COL12 -> unconnected-(A1-GPIO19-Pad25)
- A1 pad 4: ROW4 -> COL1
Routing:
- net COL0: track 76.0 -> 285.8 mm, vias 0 -> 1
- net COL1: track 76.0 -> 265.1 mm, vias 0 -> 1
- net COL2: track 76.1 -> 245.6 mm, vias 0 -> 1
- net COL3: track 76.0 -> 225.9 mm, vias 0 -> 1
- net COL4: track 76.0 -> 207.0 mm, vias 0 -> 1
- net COL5: track 76.0 -> 189.7 mm, vias 0 -> 1
- net COL6: track 76.0 -> 170.2 mm, vias 0 -> 1
- net COL7: track 76.0 -> 150.6 mm, vias 0 -> 1
- net COL8: track 76.0 -> 131.3 mm, vias 0 -> 1
- net ROW0: track 212.7 -> 264.4 mm
- net COL9: track 76.0 -> 112.9 mm, vias 0 -> 1
- net ROW4: track 174.5 -> 205.1 mm
- net ROW2: track 174.7 -> 204.0 mm
- net ROW3: track 174.5 -> 203.5 mm
- net ROW1: track 212.5 -> 235.4 mm
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
Commit message: Mounting holes and copper fill
Routing:
- added copper zone on B.Cu, net (none)
- added copper zone on F.Cu, net (none)
Other:
- outline, holes or cut-outs redrawn
Changed lines of the file:
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@@
+		(layer "Edge.Cuts")
+	)
+	(gr_circle
+		(center 106 88.1)
+		(end 106 87)
+		(stroke
+			(width 0.05)
+			(type default)
+		)
+		(fill no)
+		(layer "Edge.Cuts")
+	)
+	(gr_circle
+		(center 49 69)
+		(end 49 67.9)
+		(stroke
+			(width 0.05)
+			(type default)
+		)
+		(fill no)
+		(layer "Edge.Cuts")
+	)
+	(gr_circle
+		(center 182 88)
+		(end 182 86.9)
+		(stroke
+			(width 0.05)
+			(type default)
+		)
+		(fill no)
+		(layer "Edge.Cuts")
+	)
+	(gr_circle
+		(center 106 126)
+		(end 106 124.9)
+		(stroke
+			(width 0.05)
+			(type default)
+		)
+		(fill no)
 		(layer "Edge.Cuts")
 	)
@@
 		(layer "Edge.Cuts")
 	)
+	(gr_circle
+		(center 182 126)
+		(end 182 124.9)
+		(stroke
+			(width 0.05)
+			(type default)
+		)
+		(fill no)
+		(layer "Edge.Cuts")
+	)
+	(gr_circle
+		(center 49 126)
+		(end 49 124.9)
+		(stroke
+			(width 0.05)
+			(type default)
+		)
+		(fill no)
+		(layer "Edge.Cuts")
+	)
+	(gr_circle
+		(center 258 126)
+		(end 258 124.9)
+		(stroke
+			(width 0.05)
+			(type default)
+		)
+		(fill no)
+		(layer "Edge.Cuts")
+	)
+	(gr_circle
+		(center 242 76)
+		(end 242 74.9)
+		(stroke
+			(width 0.05)
+			(type default)
+		)
+		(fill no)
+		(layer "Edge.Cuts")
+	)
 	(gr_line
 		(start 275.5 143.5)
@@
 		(net 98)
 	)
+	(zone
+		(net 0)
+		(net_name "")
+		(layers "F.Cu" "B.Cu")
+		(hatch edge 0.5)
+		(connect_pads
+			(clearance 0.5)
+		)
+		(min_thickness 0.25)
+		(filled_areas_thickness no)
+		(fill yes
+			(thermal_gap 0.5)
+			(thermal_bridge_width 0.5)
+			(island_removal_mode 1)
+			(island_area_min 10)
+		)
+		(polygon
+			(pts
+				(xy 25 45) (xy 280 45) (xy 280 150) (xy 25 150)
+			)
+		)
+	)
 	(embedded_fonts no)
