File: kicad/keyboard/keyboard.kicad_pcb (KiCad board)
At the start: 2 copper layers, 244 x 92 mm, 119 parts, among them SW1 SW_MX, SW10 SW_MX, SW11 SW_MX, SW12 SW_MX, SW13 SW_MX, SW14 SW_MX, SW15 SW_MX, SW16 SW_MX, SW17 SW_MX, SW18 SW_MX, SW19 SW_MX, SW2 SW_MX, SW20 SW_MX, SW21 SW_MX, SW22 SW_MX, SW23 SW_MX, SW24 SW_MX, SW25 SW_MX, SW26 SW_MX, SW27 SW_MX, SW28 SW_MX, SW29 SW_MX, SW3 SW_MX, SW30 SW_MX, SW31 SW_MX, SW32 SW_MX, SW33 SW_MX, SW34 SW_MX, SW35 SW_MX, SW36 SW_MX, SW37 SW_MX, SW38 SW_MX, SW39 SW_MX, SW4 SW_MX, SW40 SW_MX, SW41 SW_MX, SW42 SW_MX, SW43 SW_MX, SW44 SW_MX, SW45 SW_MX, SW46 SW_MX, SW47 SW_MX, SW48 SW_MX, SW49 SW_MX, SW5 SW_MX, SW50 SW_MX, SW51 SW_MX, SW52 SW_MX, SW53 SW_MX, SW54 SW_MX, SW55 SW_MX, SW56 SW_MX, SW57 SW_MX, SW58 SW_MX, SW59 SW_MX, SW6 SW_MX, SW7 SW_MX, SW8 SW_MX, SW9 SW_MX

Commit message: Add licenses
Other:
- board text added: "Copyright © 2026 Jakub Świniarski"
- board text added: "Copyright © 2026 Jakub Świniarski SPDX-License-Identifier: CERN-OHL-S-2.0"
Changed lines of the file:
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@@
 		(layer "Edge.Cuts")
+	)
+	(gr_text "Copyright © 2026 Jakub Świniarski"
+		(at 271 90 270)
+		(layer "B.SilkS")
+		(effects
+			(font
+				(size 1 1)
+				(thickness 0.1)
+			)
+			(justify left bottom mirror)
+		)
+	)
+	(gr_text "Copyright © 2026 Jakub Świniarski\n\nSPDX-License-Identifier: CERN-OHL-S-2.0"
+		(at 230.5 176 0)
+		(layer "User.1")
+		(effects
+			(font
+				(size 1 1)
+				(thickness 0.125)
+			)
+			(justify bottom)
+		)
 	)
 	(segment

Commit message: Add project name silkscreen and move copyright silkscreen
Other:
- board text added: "Crude-59"
Changed lines of the file:
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@@
 		(tags "module usb pcb antenna")
 		(property "Reference" "A1"
-			(at 8.89 25.1 90)
+			(at 8.89 18.8175 270)
 			(unlocked yes)
 			(layer "F.SilkS")
@@
 		)
 		(fp_text user "${REFERENCE}"
-			(at 8.89 24.13 90)
+			(at 8.89 19.505 270)
 			(layer "F.Fab")
 			(effects
@@
 	)
 	(gr_text "Copyright © 2026 Jakub Świniarski"
-		(at 271 90 270)
+		(at 259.5 60.5 90)
+		(layer "B.SilkS")
+		(effects
+			(font
+				(size 1 1)
+				(thickness 0.1)
+			)
+			(justify left bottom mirror)
+		)
+	)
+	(gr_text "Crude-59"
+		(at 256.5 71 90)
 		(layer "B.SilkS")
 		(effects

Commit message: Update copyright notices
Other:
- board text added: "Crude-59 © 2026 Jakub Świniarski"
- board text added: "© 2026 Jakub Świniarski SPDX-License-Identifier: CERN-OHL-S-2.0"
- board text removed: "Copyright © 2026 Jakub Świniarski"
- board text removed: "Copyright © 2026 Jakub Świniarski SPDX-License-Identifier: CERN-OHL-S-2.0"
- board text removed: "Crude-59"
Changed lines of the file:
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@@
 		(layer "Edge.Cuts")
 	)
-	(gr_text "Copyright © 2026 Jakub Świniarski"
-		(at 259.5 60.5 90)
+	(gr_text "Crude-59\n\n© 2026 Jakub Świniarski"
+		(at 259.5 75 90)
 		(layer "B.SilkS")
 		(effects
@@
 				(thickness 0.1)
 			)
-			(justify left bottom mirror)
+			(justify bottom mirror)
 		)
 	)
-	(gr_text "Crude-59"
-		(at 256.5 71 90)
-		(layer "B.SilkS")
-		(effects
-			(font
-				(size 1 1)
-				(thickness 0.1)
-			)
-			(justify left bottom mirror)
-		)
-	)
-	(gr_text "Copyright © 2026 Jakub Świniarski\n\nSPDX-License-Identifier: CERN-OHL-S-2.0"
+	(gr_text "© 2026 Jakub Świniarski\n\nSPDX-License-Identifier: CERN-OHL-S-2.0"
 		(at 230.5 176 0)
 		(layer "User.1")
