File: kicad/keyboard/keyboard.kicad_sch (KiCad schematic)
At the start: 119 parts, among them SW1 SW_MX, SW10 SW_MX, SW11 SW_MX, SW12 SW_MX, SW13 SW_MX, SW14 SW_MX, SW15 SW_MX, SW16 SW_MX, SW17 SW_MX, SW18 SW_MX, SW19 SW_MX, SW2 SW_MX, SW20 SW_MX, SW21 SW_MX, SW22 SW_MX, SW23 SW_MX, SW24 SW_MX, SW25 SW_MX, SW26 SW_MX, SW27 SW_MX, SW28 SW_MX, SW29 SW_MX, SW3 SW_MX, SW30 SW_MX, SW31 SW_MX, SW32 SW_MX, SW33 SW_MX, SW34 SW_MX, SW35 SW_MX, SW36 SW_MX, SW37 SW_MX, SW38 SW_MX, SW39 SW_MX, SW4 SW_MX, SW40 SW_MX, SW41 SW_MX, SW42 SW_MX, SW43 SW_MX, SW44 SW_MX, SW45 SW_MX, SW46 SW_MX, SW47 SW_MX, SW48 SW_MX, SW49 SW_MX, SW5 SW_MX, SW50 SW_MX, SW51 SW_MX, SW52 SW_MX, SW53 SW_MX, SW54 SW_MX, SW55 SW_MX, SW56 SW_MX, SW57 SW_MX, SW58 SW_MX, SW59 SW_MX, SW6 SW_MX, SW7 SW_MX, SW8 SW_MX, SW9 SW_MX

Commit message: Add licenses
Other:
- note added: "Copyright © 2026 Jakub Świniarski SPDX-License-Identifier: CERN-OHL-S-2.0"
Changed lines of the file:
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@@
 	(generator_version "9.0")
 	(paper "A4")
+	(text "Copyright © 2026 Jakub Świniarski\n\nSPDX-License-Identifier: CERN-OHL-S-2.0"
+		(exclude_from_sim no)
+		(at 232.664 173.482 0)
+		(effects
+			(font
+				(size 1.27 1.27)
+			)
+		)
+	)
 	(junction
 		(at 139.7 114.3)

Commit message: Update copyright notices
Other:
- note added: "© 2026 Jakub Świniarski SPDX-License-Identifier: CERN-OHL-S-2.0"
- note removed: "Copyright © 2026 Jakub Świniarski SPDX-License-Identifier: CERN-OHL-S-2.0"
Changed lines of the file:
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@@
 	(generator_version "9.0")
 	(paper "A4")
-	(text "Copyright © 2026 Jakub Świniarski\n\nSPDX-License-Identifier: CERN-OHL-S-2.0"
+	(text "© 2026 Jakub Świniarski\n\nSPDX-License-Identifier: CERN-OHL-S-2.0"
 		(exclude_from_sim no)
 		(at 232.664 173.482 0)
